File: hardware/LED_ring.kicad_sch (KiCad schematic)
At the start: 62 parts, among them U1 MAX7221xWG

Commit message: start layout, finalize schematic
Parts:
- C201: renamed from C1; footprint (none) -> Capacitor_SMD:C_0805_2012Metric
- D201: renamed from D1; footprint (none) -> LED_SMD:LED_0603_1608Metric
- D202: renamed from D9; footprint (none) -> LED_SMD:LED_0603_1608Metric
- D203: renamed from D17; footprint (none) -> LED_SMD:LED_0603_1608Metric
- D204: renamed from D25; footprint (none) -> LED_SMD:LED_0603_1608Metric
- D205: renamed from D32; footprint (none) -> LED_SMD:LED_0603_1608Metric
- D206: renamed from D39; footprint (none) -> LED_SMD:LED_0603_1608Metric
- D207: renamed from D46; footprint (none) -> LED_SMD:LED_0603_1608Metric
- D208: renamed from D53; footprint (none) -> LED_SMD:LED_0603_1608Metric
- D209: renamed from D2; footprint (none) -> LED_SMD:LED_0603_1608Metric
- D210: renamed from D10; footprint (none) -> LED_SMD:LED_0603_1608Metric
- D211: renamed from D18; footprint (none) -> LED_SMD:LED_0603_1608Metric
- D212: renamed from D26; footprint (none) -> LED_SMD:LED_0603_1608Metric
- D213: renamed from D33; footprint (none) -> LED_SMD:LED_0603_1608Metric
- D214: renamed from D40; footprint (none) -> LED_SMD:LED_0603_1608Metric
- D215: renamed from D47; footprint (none) -> LED_SMD:LED_0603_1608Metric
- D216: renamed from D54; footprint (none) -> LED_SMD:LED_0603_1608Metric
- D217: renamed from D3; footprint (none) -> LED_SMD:LED_0603_1608Metric
- D218: renamed from D11; footprint (none) -> LED_SMD:LED_0603_1608Metric
- D219: renamed from D19; footprint (none) -> LED_SMD:LED_0603_1608Metric
- D220: renamed from D27; footprint (none) -> LED_SMD:LED_0603_1608Metric
- D221: renamed from D34; footprint (none) -> LED_SMD:LED_0603_1608Metric
- D222: renamed from D41; footprint (none) -> LED_SMD:LED_0603_1608Metric
- D223: renamed from D48; footprint (none) -> LED_SMD:LED_0603_1608Metric
- D224: renamed from D55; footprint (none) -> LED_SMD:LED_0603_1608Metric
- D225: renamed from D4; footprint (none) -> LED_SMD:LED_0603_1608Metric
- D226: renamed from D12; footprint (none) -> LED_SMD:LED_0603_1608Metric
- D227: renamed from D20; footprint (none) -> LED_SMD:LED_0603_1608Metric
- D228: renamed from D28; footprint (none) -> LED_SMD:LED_0603_1608Metric
- D229: renamed from D35; footprint (none) -> LED_SMD:LED_0603_1608Metric
- D230: renamed from D42; footprint (none) -> LED_SMD:LED_0603_1608Metric
- D231: renamed from D49; footprint (none) -> LED_SMD:LED_0603_1608Metric
- D232: renamed from D56; footprint (none) -> LED_SMD:LED_0603_1608Metric
- D233: renamed from D5; footprint (none) -> LED_SMD:LED_0603_1608Metric
- D234: renamed from D13; footprint (none) -> LED_SMD:LED_0603_1608Metric
- D235: renamed from D21; footprint (none) -> LED_SMD:LED_0603_1608Metric
- D236: renamed from D29; footprint (none) -> LED_SMD:LED_0603_1608Metric
- D237: renamed from D36; footprint (none) -> LED_SMD:LED_0603_1608Metric
- D238: renamed from D43; footprint (none) -> LED_SMD:LED_0603_1608Metric
- D239: renamed from D50; footprint (none) -> LED_SMD:LED_0603_1608Metric
- D240: renamed from D57; footprint (none) -> LED_SMD:LED_0603_1608Metric
- D241: renamed from D6; footprint (none) -> LED_SMD:LED_0603_1608Metric
- D242: renamed from D14; footprint (none) -> LED_SMD:LED_0603_1608Metric
- D243: renamed from D22; footprint (none) -> LED_SMD:LED_0603_1608Metric
- D244: renamed from D30; footprint (none) -> LED_SMD:LED_0603_1608Metric
- D245: renamed from D37; footprint (none) -> LED_SMD:LED_0603_1608Metric
- D246: renamed from D44; footprint (none) -> LED_SMD:LED_0603_1608Metric
- D247: renamed from D51; footprint (none) -> LED_SMD:LED_0603_1608Metric
- D248: renamed from D58; footprint (none) -> LED_SMD:LED_0603_1608Metric
- D249: renamed from D7; footprint (none) -> LED_SMD:LED_0603_1608Metric
- D250: renamed from D15; footprint (none) -> LED_SMD:LED_0603_1608Metric
- D251: renamed from D23; footprint (none) -> LED_SMD:LED_0603_1608Metric
- D252: renamed from D31; footprint (none) -> LED_SMD:LED_0603_1608Metric
- D253: renamed from D38; footprint (none) -> LED_SMD:LED_0603_1608Metric
- D254: renamed from D45; footprint (none) -> LED_SMD:LED_0603_1608Metric
- D255: renamed from D52; footprint (none) -> LED_SMD:LED_0603_1608Metric
- D256: renamed from D59; footprint (none) -> LED_SMD:LED_0603_1608Metric
- D257: renamed from D8; footprint (none) -> LED_SMD:LED_0603_1608Metric
- D258: renamed from D16; footprint (none) -> LED_SMD:LED_0603_1608Metric
- D259: renamed from D24; footprint (none) -> LED_SMD:LED_0603_1608Metric
- R201: renamed from R1; footprint (none) -> Resistor_SMD:R_0805_2012Metric
- renumbered U1 to U201
