File: hardware/dcf77.kicad_pcb (KiCad board)
At the start: 4 copper layers, 150 x 150 mm, 312 parts, among them J501 Jack-DC, J502 DCF77 Antenna, J503 SWD, J504 USB_B, Q401 BSS138, Q402 BSS138, Q403 BSS138, Q404 BSS138, Q405 BSS138, Q406 BSS138, Q407 BSS138, Q408 BSS138, Q409 BSS138, Q410 BSS138, Q411 BSS138, Q412 BSS138, Q413 BSS138, Q501 BSS138, Q502 BSS138, Q503 BSS138, Q504 BSS138, Q505 BSS138, Q506 BSS138, Q507 BSS138, Q508 BC856, Q509 BSS138, Q510 BSS138, Q511 BSS138, U201 MAX7221xWG, U301 MAX7221xWG, U401 74HC595, U402 MAX7221xWG, U403 MAX7221xWG, U404 74HC595, U405 MAX7221xWG, U501 L7805, U502 AZ1117-3.3, U503 STM32F103C8Tx, Y501 8MHz, Y502 32.768kHz

Commit message: update Layout
Parts:
- moved D233 80.3 mm to (65.2, 157.5), turned to 102 degrees
- moved D255 72.9 mm to (74.7, 112.8), turned to -126 degrees
- moved D232 69.2 mm to (62.6, 157.9), turned to 96 degrees
- moved D234 67.7 mm to (67.7, 156.8), turned to 108 degrees
- moved D237 61.6 mm to (74.7, 153.2), turned to 126 degrees
- moved D258 61.4 mm to (67.7, 109.2), turned to -108 degrees
- moved D252 61.0 mm to (80.2, 118.3), turned to -144 degrees
- moved D245 60.7 mm to (84.9, 135.6), turned to 174 degrees
- moved D235 59.3 mm to (70.2, 155.8), turned to 114 degrees
- moved D257 58.2 mm to (70.2, 110.1), turned to -114 degrees
- moved D236 57.7 mm to (72.5, 154.6), turned to 120 degrees
- moved D247 56.3 mm to (84.9, 130.4), turned to -174 degrees
- moved D241 55.8 mm to (81.6, 145.5), turned to 150 degrees
- moved D239 54.9 mm to (78.6, 149.7), turned to 138 degrees
- moved D238 51.6 mm to (76.7, 151.6), turned to 132 degrees
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
Commit message: update Layout
Parts:
- AFF401, AFF402, AFF403, AFF404, AFF405, AFF406, AFF407, AFF408, AFF409, AFF410, AFF411, AFF412, AFF413, AFF414, AFF415, AFF416, AFF417, AFF418, AFF419, AFF420: footprint Display_7Segment:7SegmentLED_LTS6760_LTS6780 -> eigene:7_Segment_SMD; moved to B.Cu
- C201, C301, R201, R301: moved to F.Cu
- D401, D402, D403, D404, D405, D406, D407, D408, D409, D410, D411, D412, D413, D503: moved to B.Cu
- moved D412 296.9 mm to (59.5, 157.5), turned to 180 degrees
- moved D408 294.3 mm to (59.5, 142.2), turned to 180 degrees
- moved D406 286.1 mm to (72.2, 161.3), turned to 180 degrees
- moved D413 280.6 mm to (59.5, 161.3), turned to 180 degrees
- moved D405 268.6 mm to (72.2, 157.5), turned to 180 degrees
- moved AFF410 260.1 mm to (42.8, 78.7), turned to 180 degrees
- moved AFF418 256.6 mm to (42.8, 132.1), turned to 180 degrees
- moved D407 251.6 mm to (72.2, 165.1), turned to 180 degrees
- moved D403 249.1 mm to (72.2, 149.9), turned to 180 degrees
- moved D404 245.9 mm to (72.2, 153.7), turned to 180 degrees
- moved D411 237.1 mm to (59.5, 153.7), turned to 180 degrees
- moved D409 230.8 mm to (59.5, 146.1), turned to 180 degrees
- moved AFF413 228.2 mm to (58.1, 105.4), turned to 180 degrees
- moved AFF412 224.5 mm to (35.2, 78.7), turned to 180 degrees
- moved U405 224.0 mm to (65.4, 123.2)
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Routing:
- net Net-(D203-Pad2): track 0.00 -> 151.3 mm, vias 0 -> 8
- net Net-(D201-Pad2): track 0.00 -> 149.0 mm, vias 0 -> 8
- net Net-(D202-Pad2): track 0.00 -> 146.9 mm, vias 0 -> 8
- net Net-(D208-Pad2): track 0.00 -> 139.9 mm, vias 0 -> 7
- net Net-(D206-Pad2): track 0.00 -> 138.0 mm, vias 0 -> 7
- net Net-(D204-Pad2): track 0.00 -> 135.9 mm, vias 0 -> 7
- net Net-(D207-Pad2): track 0.00 -> 133.9 mm, vias 0 -> 7
- net Net-(D205-Pad2): track 0.00 -> 132.0 mm, vias 0 -> 7
- net Net-(D333-Pad1): track 0.00 -> 22.1 mm
- net Net-(D317-Pad1): track 0.00 -> 21.4 mm
- net Net-(D301-Pad1): track 0.00 -> 21.4 mm
- net Net-(D349-Pad1): track 0.00 -> 21.4 mm
- net Net-(D309-Pad1): track 0.00 -> 21.4 mm
- net Net-(D341-Pad1): track 0.00 -> 21.4 mm
- net Net-(D325-Pad1): track 0.00 -> 21.3 mm
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Other:
- board text added: "0"
- board text added: "1"
- board text added: "10"
- board text added: "2"
- board text added: "20"
- board text added: "30"
- board text added: "4"
- board text added: "40"
- board text added: "50"
- board text added: "8"
- board text added: "80"
- board text added: "ANTENNE"
- board text added: "BIT-NR."
- board text added: "CEST"
- board text added: "CET"
- board text added: "DATUM"
- board text added: "DCF77"
- board text added: "DI"
- board text added: "DO"
- board text added: "FR"
- board text added: "JAHR"
- board text added: "METEO DATA"
- board text added: "MI"
- board text added: "MINUTE"
- board text added: "MO"
- board text added: "MONAT"
- board text added: "P1"
- board text added: "P2"
- board text added: "P3"
- board text added: "PERIODENDAUER"
- board text added: "PULSLÄNGE"
- board text added: "Parity Bit 1"
- board text added: "Parity Bit 2"
- board text added: "Parity Bit 3"
- board text added: "Parity Error"
- board text added: "RTC Sync"
- board text added: "SA"
- board text added: "SCHALTSEKUNDE"
- board text added: "SCHALTSTUNDE"
- board text added: "SO"
- board text added: "START"
- board text added: "STUNDE"
- board text added: "TAG"
- board text added: "UHRZEIT"
- board text added: "WOCHENTAG"
- board text removed: "Signal"

Commit message: update Schematic
Parts:
- moved C301 175.3 mm to (59.9, 122.3)
- moved R301 175.3 mm to (60.1, 117.1)
- moved U301 174.8 mm to (71.1, 120.0)
- moved U401 120.4 mm to (99.7, 61.0)
- moved U404 99.9 mm to (99.7, 73.0)
- moved C201 52.1 mm to (123.5, 70.5)
- moved R201 51.0 mm to (124.1, 74.0)
- moved U201 48.6 mm to (113.7, 75.6)
- moved U405 23.6 mm to (71.1, 100.3)
- moved U503 12.7 mm to (118.7, 47.0)
- moved D401 9.22 mm to (63.0, 142.2)
- moved D402 9.22 mm to (63.0, 146.1)
- moved D403 9.22 mm to (63.0, 149.9)
- moved D404 9.22 mm to (63.0, 153.7)
- moved D405 9.22 mm to (63.0, 157.5)
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Connections:
- Y502 pad 2: Net-(C511-Pad1) -> unconnected-(Y502-Pad2)
- Y502 pad 3: (no net) -> unconnected-(Y502-Pad3)
- Y502 pad 4: (no net) -> Net-(C511-Pad1)
Routing:
- net Net-(D308-Pad2): track 0.00 -> 265.9 mm, vias 0 -> 7
- net Net-(D307-Pad2): track 0.00 -> 253.7 mm, vias 0 -> 7
- net Net-(D306-Pad2): track 0.00 -> 241.2 mm, vias 0 -> 7
- net Net-(D303-Pad2): track 0.00 -> 238.8 mm, vias 0 -> 8
- net Net-(D305-Pad2): track 0.00 -> 229.3 mm, vias 0 -> 7
- net Net-(D302-Pad2): track 0.00 -> 225.3 mm, vias 0 -> 8
- net Net-(D304-Pad2): track 0.00 -> 216.9 mm, vias 0 -> 7
- net Net-(D301-Pad2): track 0.00 -> 211.1 mm, vias 0 -> 8
- net Net-(AFF401-Pad6): track 0.00 -> 88.8 mm, vias 0 -> 8
- net Net-(AFF401-Pad7): track 0.00 -> 84.9 mm, vias 0 -> 8
- net Net-(AFF401-Pad1): track 0.00 -> 79.9 mm, vias 0 -> 7
- net Net-(AFF411-Pad3): track 0.00 -> 79.9 mm, vias 0 -> 3
- net Net-(AFF401-Pad4): track 0.00 -> 78.7 mm, vias 0 -> 8
- net Net-(AFF401-Pad9): track 0.00 -> 75.8 mm, vias 0 -> 7
- net Net-(AFF401-Pad2): track 0.00 -> 75.3 mm, vias 0 -> 8
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Other:
- outline, holes or cut-outs redrawn
- board text added: "Antenne"

Commit message: update
Parts:
- C503, C517: footprint Capacitor_SMD:C_0805_2012Metric -> Capacitor_SMD:CP_Elec_5x5.8
- C518: value C -> 100n
- FB501, FB502: footprint Resistor_SMD:R_4020_10251Metric -> eigene:SMB-001
- moved R510 170.8 mm to (104.0, 53.8), turned to 180 degrees
- moved R517 166.5 mm to (120.1, 36.8), turned to 180 degrees
- moved C512 166.2 mm to (101.2, 44.7), turned to 180 degrees
- moved R523 165.4 mm to (121.9, 30.7), turned to 180 degrees
- moved R516 162.8 mm to (119.1, 30.0), turned to -90 degrees
- moved C510 160.3 mm to (105.8, 55.9), turned to 180 degrees
- moved C509 157.9 mm to (102.2, 55.9)
- moved C511 153.7 mm to (106.3, 44.7)
- moved R527 150.1 mm to (131.8, 39.6), turned to 90 degrees
- moved Q505 148.7 mm to (120.1, 33.8), turned to 90 degrees
- moved Y502 148.0 mm to (103.8, 48.8), turned to 180 degrees
- moved C516 147.2 mm to (136.1, 31.5), turned to -90 degrees
- moved C515 146.0 mm to (136.1, 26.9), turned to 90 degrees
- moved R525 145.5 mm to (133.9, 39.6), turned to -90 degrees
- moved R530 139.7 mm to (140.0, 40.6), turned to 90 degrees
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Connections:
- C518 pad 1: +3.3V -> +3V3
- D501 pad 2: +3.3V -> +3V3
- J502 pad 4: +3.3V -> +3V3
- J503 pad 1: +3.3V -> +3V3
- Q504 pad 1: +3.3V -> +3V3
- Q506 pad 1: +3.3V -> +3V3
- R503 pad 2: +3.3V -> +3V3
- R513 pad 2: +3.3V -> +3V3
- R519 pad 2: +3.3V -> +3V3
- R523 pad 1: +3.3V -> +3V3
- U503 pad 24: +3.3V -> +3V3
- U503 pad 36: +3.3V -> +3V3
- U503 pad 48: +3.3V -> +3V3
- U503 pad 9: +3.3V -> +3V3
- Y502 pad 1: Net-(C512-Pad1) -> Net-(C511-Pad1)
- Y502 pad 4: Net-(C511-Pad1) -> Net-(C512-Pad1)
Routing:
- net Net-(AFF411-Pad3): track 79.9 -> 10.6 mm, vias 3 -> 0
- net Net-(AFF409-Pad3): track 62.5 -> 10.6 mm, vias 3 -> 0
- net Net-(AFF407-Pad3): track 58.4 -> 10.6 mm, vias 3 -> 0
- net GND: track 0.00 -> 38.0 mm, vias 0 -> 31
- net Net-(AFF405-Pad3): track 48.1 -> 10.6 mm, vias 3 -> 0
- net Net-(AFF403-Pad3): track 46.3 -> 11.4 mm, vias 1 -> 0
- net USB+: track 0.00 -> 33.0 mm
- net USB-: track 0.00 -> 30.8 mm
- net Net-(AFF401-Pad6): track 88.8 -> 64.9 mm, vias 8 -> 6
- net /Disconnect: track 0.00 -> 23.7 mm
- net Net-(AFF401-Pad4): track 78.7 -> 58.4 mm, vias 8 -> 6
- net Net-(AFF401-Pad7): track 84.9 -> 64.7 mm, vias 8 -> 7
- net Net-(AFF401-Pad5): track 74.1 -> 54.2 mm, vias 8 -> 6
- net Net-(AFF401-Pad9): track 75.8 -> 56.4 mm, vias 7 -> 6
- net Net-(C509-Pad1): track 0.00 -> 18.5 mm
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- added copper zone on F.Cu, net +3V3
- added copper zone on In2.Cu, net +3V3
- added copper zone on F.Cu, net +5V
- added copper zone on In2.Cu, net +5V
- added copper zone on F.Cu, net GND
- added copper zone on In1.Cu, net GND
- added copper zone on F.Cu, net Net-(C503-Pad1)
- added copper zone on F.Cu, net VBUS
Other:
- outline, holes or cut-outs redrawn
- board text added: "3V3 SWIO SWCLK GND"
- board text added: "BIT-VAL"
- board text added: "JLCJLCJLCJLC"
- board text removed: "BIT-NR."

Commit message: update
Parts:
- moved Q406 231.0 mm to (56.9, 161.3), turned to 180 degrees
- moved R435 227.4 mm to (59.9, 153.7), turned to 90 degrees
- moved R408 226.3 mm to (52.3, 142.2), turned to 180 degrees
- moved R407 225.8 mm to (68.1, 165.1), turned to 180 degrees
- moved R442 218.9 mm to (63.2, 118.6), turned to -90 degrees
- moved R438 217.6 mm to (62.0, 149.9), turned to -90 degrees
- moved R405 217.6 mm to (68.1, 157.5), turned to 180 degrees
- moved R413 217.6 mm to (52.3, 161.3), turned to 180 degrees
- moved R441 215.0 mm to (59.9, 146.1), turned to 90 degrees
- moved R532 212.4 mm to (59.9, 165.1), turned to -90 degrees
- moved R426 208.4 mm to (77.7, 149.9), turned to -90 degrees
- moved R410 207.8 mm to (52.3, 149.9), turned to 180 degrees
- moved R439 207.7 mm to (59.9, 149.9), turned to 90 degrees
- moved Q401 206.5 mm to (56.9, 142.2), turned to 180 degrees
- moved R420 206.4 mm to (77.7, 157.5), turned to -90 degrees
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Connections:
- C521 pad 1: +3V3 -> +5V
- D504 pad 1: Net-(D504-Pad1) -> Net-(R526-Pad2)
- D504 pad 2: Net-(D504-Pad2) -> +5V
- Q510 pad 3: Net-(D504-Pad1) -> Net-(R526-Pad1)
- R526 pad 1: Net-(D504-Pad2) -> Net-(R526-Pad1)
- R526 pad 2: +5V -> Net-(R526-Pad2)
Routing:
- net GND: track 38.0 -> 173.3 mm, vias 31 -> 80
- net Net-(AFF402-Pad6): track 0.00 -> 72.4 mm, vias 0 -> 7
- net Net-(AFF402-Pad5): track 0.00 -> 71.4 mm, vias 0 -> 7
- net Net-(AFF402-Pad7): track 0.00 -> 68.9 mm, vias 0 -> 8
- net Net-(AFF402-Pad4): track 0.00 -> 67.0 mm, vias 0 -> 8
- net Net-(AFF402-Pad2): track 0.00 -> 64.6 mm, vias 0 -> 7
- net Net-(AFF402-Pad9): track 0.00 -> 63.8 mm, vias 0 -> 8
- net Net-(AFF402-Pad1): track 0.00 -> 59.7 mm, vias 0 -> 8
- net Net-(AFF402-Pad10): track 0.00 -> 58.4 mm, vias 0 -> 6
- net /CPU/SER_Latch: track 0.00 -> 53.4 mm, vias 0 -> 4
- net /CPU/SER_CLK: track 0.00 -> 52.0 mm, vias 0 -> 3
- net +3V3: track 13.5 -> 59.9 mm, vias 12 -> 24
- net +5V: track 15.1 -> 54.4 mm, vias 17 -> 34
- net /CPU/SER_Data: track 0.00 -> 35.9 mm, vias 0 -> 2
- net Net-(D233-Pad1): track 18.9 -> 53.9 mm, vias 0 -> 1
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- added copper zone on F.Cu, net Net-(D502-Pad2)
Other:
- outline, holes or cut-outs redrawn
