File: hardware/Status.kicad_sch (KiCad schematic)
At the start: 87 parts, among them Q1 BSS138, Q10 BSS138, Q11 BSS138, Q12 BSS138, Q13 BSS138, Q2 BSS138, Q3 BSS138, Q4 BSS138, Q5 BSS138, Q6 BSS138, Q7 BSS138, Q8 BSS138, Q9 BSS138, U3 MAX7221xWG, U4 MAX7221xWG, U5 74HC595, U6 74HC595

Commit message: start layout, finalize schematic
Parts:
- added AFF413, AFF414, AFF415, AFF416, AFF417, AFF418, AFF419, AFF420: LTS-6980HR, Display_7Segment:7SegmentLED_LTS6760_LTS6780, symbol Display_Character:LTS-6980HR
- added R442: 20k, Resistor_SMD:R_0805_2012Metric, symbol Device:R
- added U405: MAX7221xWG, Package_SO:SOIC-24W_7.5x15.4mm_P1.27mm, symbol Driver_LED:MAX7221xWG
- C401: renamed from C3; footprint (none) -> Capacitor_SMD:C_0805_2012Metric
- C402: renamed from C4; footprint (none) -> Capacitor_SMD:C_0805_2012Metric
- C403: renamed from C5; footprint (none) -> Capacitor_SMD:C_0805_2012Metric
- C404: renamed from C6; footprint (none) -> Capacitor_SMD:C_0805_2012Metric
- D401: renamed from D119; footprint (none) -> LED_SMD:LED_0603_1608Metric
- D402: renamed from D120; footprint (none) -> LED_SMD:LED_0603_1608Metric
- D403: renamed from D121; footprint (none) -> LED_SMD:LED_0603_1608Metric
- D404: renamed from D122; footprint (none) -> LED_SMD:LED_0603_1608Metric
- D405: renamed from D123; footprint (none) -> LED_SMD:LED_0603_1608Metric
- D406: renamed from D124; footprint (none) -> LED_SMD:LED_0603_1608Metric
- D407: renamed from D125; footprint (none) -> LED_SMD:LED_0603_1608Metric
- D408: renamed from D126; footprint (none) -> LED_SMD:LED_0603_1608Metric
- D409: renamed from D127; footprint (none) -> LED_SMD:LED_0603_1608Metric
- D410: renamed from D128; footprint (none) -> LED_SMD:LED_0603_1608Metric
- D411: renamed from D129; footprint (none) -> LED_SMD:LED_0603_1608Metric
- D412: renamed from D130; footprint (none) -> LED_SMD:LED_0603_1608Metric
- D413: renamed from D131; footprint (none) -> LED_SMD:LED_0603_1608Metric
- R401: renamed from R5; footprint (none) -> Resistor_SMD:R_0805_2012Metric
- R402: renamed from R6; footprint (none) -> Resistor_SMD:R_0805_2012Metric
- R403: renamed from R7; footprint (none) -> Resistor_SMD:R_0805_2012Metric
- R404: renamed from R8; footprint (none) -> Resistor_SMD:R_0805_2012Metric
- R405: renamed from R9; footprint (none) -> Resistor_SMD:R_0805_2012Metric
- R406: renamed from R18; footprint (none) -> Resistor_SMD:R_0805_2012Metric
- R407: renamed from R27; footprint (none) -> Resistor_SMD:R_0805_2012Metric
- R408: renamed from R28; footprint (none) -> Resistor_SMD:R_0805_2012Metric
- R409: renamed from R29; footprint (none) -> Resistor_SMD:R_0805_2012Metric
- R410: renamed from R30; footprint (none) -> Resistor_SMD:R_0805_2012Metric
- R411: renamed from R31; footprint (none) -> Resistor_SMD:R_0805_2012Metric
- R412: renamed from R37; footprint (none) -> Resistor_SMD:R_0805_2012Metric
- R413: renamed from R43; footprint (none) -> Resistor_SMD:R_0805_2012Metric
- R414: renamed from R19; footprint (none) -> Resistor_SMD:R_0805_2012Metric
- R415: renamed from R10; footprint (none) -> Resistor_SMD:R_0805_2012Metric
- R416: renamed from R20; footprint (none) -> Resistor_SMD:R_0805_2012Metric
- R417: renamed from R11; footprint (none) -> Resistor_SMD:R_0805_2012Metric
- R418: renamed from R21; footprint (none) -> Resistor_SMD:R_0805_2012Metric
- R419: renamed from R12; footprint (none) -> Resistor_SMD:R_0805_2012Metric
- R420: renamed from R22; footprint (none) -> Resistor_SMD:R_0805_2012Metric
- R421: renamed from R13; footprint (none) -> Resistor_SMD:R_0805_2012Metric
- R422: renamed from R23; footprint (none) -> Resistor_SMD:R_0805_2012Metric
- R423: renamed from R14; footprint (none) -> Resistor_SMD:R_0805_2012Metric
- R424: renamed from R38; footprint (none) -> Resistor_SMD:R_0805_2012Metric
- R425: renamed from R32; footprint (none) -> Resistor_SMD:R_0805_2012Metric
- R426: renamed from R24; footprint (none) -> Resistor_SMD:R_0805_2012Metric
- R427: renamed from R3; footprint (none) -> Resistor_SMD:R_0805_2012Metric
- R428: renamed from R4; footprint (none) -> Resistor_SMD:R_0805_2012Metric
- R429: renamed from R15; footprint (none) -> Resistor_SMD:R_0805_2012Metric
- R430: renamed from R39; footprint (none) -> Resistor_SMD:R_0805_2012Metric
- R431: renamed from R33; footprint (none) -> Resistor_SMD:R_0805_2012Metric
- R432: renamed from R25; footprint (none) -> Resistor_SMD:R_0805_2012Metric
- R433: renamed from R16; footprint (none) -> Resistor_SMD:R_0805_2012Metric
- R434: renamed from R40; footprint (none) -> Resistor_SMD:R_0805_2012Metric
- R435: renamed from R34; footprint (none) -> Resistor_SMD:R_0805_2012Metric
- R436: renamed from R26; footprint (none) -> Resistor_SMD:R_0805_2012Metric
- R437: renamed from R17; footprint (none) -> Resistor_SMD:R_0805_2012Metric
- R438: renamed from R41; footprint (none) -> Resistor_SMD:R_0805_2012Metric
- R439: renamed from R35; footprint (none) -> Resistor_SMD:R_0805_2012Metric
- R440: renamed from R42; footprint (none) -> Resistor_SMD:R_0805_2012Metric
- R441: renamed from R36; footprint (none) -> Resistor_SMD:R_0805_2012Metric
- U401: renamed from U5; footprint (none) -> Package_SO:SO-16_3.9x9.9mm_P1.27mm
- U404: renamed from U6; footprint (none) -> Package_SO:SO-16_3.9x9.9mm_P1.27mm
- renumbered AFF1 to AFF401, AFF7 to AFF402, AFF2 to AFF403, AFF8 to AFF404, AFF3 to AFF405, AFF9 to AFF406, AFF4 to AFF407, AFF10 to AFF408, AFF5 to AFF409, AFF11 to AFF410, AFF6 to AFF411, AFF12 to AFF412, Q1 to Q401, Q2 to Q402, Q3 to Q403, Q4 to Q404, Q5 to Q405, Q9 to Q406, Q6 to Q407, Q10 to Q408, Q7 to Q409, Q11 to Q410, Q8 to Q411, Q12 to Q412, Q13 to Q413, U3 to U402, U4 to U403
Connections:
- net +5V: now also R442.1, U405.19 (V+)
- net CLK: now also U405.13 (CLK)
- net Data: now also U405.1 (DIN)
- net GND: now also U405.4 (GND), U405.9 (GND)
- new net: AFF413.3 (C.K.), AFF413.8 (C.K.), U405.2 (DIG_0)
- new net: AFF413.5 (DP), AFF414.5 (DP), AFF415.5 (DP), U405.22 (SEG_DP)
- new net: AFF414.3 (C.K.), AFF414.8 (C.K.), U405.11 (DIG_1)
- new net: AFF418.3 (C.K.), AFF418.8 (C.K.), U405.10 (DIG_5)
- new net: AFF415.7 (a), AFF416.7 (a), AFF417.7 (a), AFF418.7 (a), AFF419.7 (a), AFF420.7 (a), U405.14 (SEG_A)
- new net: AFF415.9 (f), AFF416.9 (f), AFF417.9 (f), AFF418.9 (f), AFF419.9 (f), AFF420.9 (f), U405.15 (SEG_F)
- new net: AFF415.6 (b), AFF416.6 (b), AFF417.6 (b), AFF418.6 (b), AFF419.6 (b), AFF420.6 (b), U405.16 (SEG_B)
- new net: AFF415.10 (g), AFF416.10 (g), AFF417.10 (g), AFF418.10 (g), AFF419.10 (g), AFF420.10 (g), U405.17 (SEG_G)
- new net: R442.2, U405.18 (ISET)
- new net: AFF415.4 (c), AFF416.4 (c), AFF417.4 (c), AFF418.4 (c), AFF419.4 (c), AFF420.4 (c), U405.20 (SEG_C)
- new net: AFF415.1 (e), AFF416.1 (e), AFF417.1 (e), AFF418.1 (e), AFF419.1 (e), AFF420.1 (e), U405.21 (SEG_E)
- new net: AFF415.2 (d), AFF416.2 (d), AFF417.2 (d), AFF418.2 (d), AFF419.2 (d), AFF420.2 (d), U405.23 (SEG_D)
- new net: AFF417.3 (C.K.), AFF417.8 (C.K.), U405.3 (DIG_4)
- new net: AFF419.3 (C.K.), AFF419.8 (C.K.), U405.5 (DIG_6)
- new net: AFF415.3 (C.K.), AFF415.8 (C.K.), U405.6 (DIG_2)
- new net: AFF416.3 (C.K.), AFF416.8 (C.K.), U405.7 (DIG_3)
- new net: AFF420.3 (C.K.), AFF420.8 (C.K.), U405.8 (DIG_7)
- new net /CS_pulse: U405.12 (~{CS})
- no-connect marks 10 -> 11
Other:
- moved on the sheet: C401, C402, C403, C404, D401, D402, D403, D404, D405, D406, D407, D408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

Commit message: update Layout
Parts:
- AFF401, AFF402, AFF403, AFF404, AFF405, AFF406, AFF407, AFF408, AFF409, AFF410, AFF411, AFF412, AFF413, AFF414, AFF415, AFF416, AFF417, AFF418, AFF419, AFF420: footprint Display_7Segment:7SegmentLED_LTS6760_LTS6780 -> eigene:7_Segment_SMD
Changed lines of the file:
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@@
     (property "Reference" "AFF402" (id 0) (at 208.28 39.4802 0))
     (property "Value" "LTS-6980HR" (id 1) (at 208.28 42.0171 0))
-    (property "Footprint" "Display_7Segment:7SegmentLED_LTS6760_LTS6780" (id 2) (at 208.28 71.12 0)
+    (property "Footprint" "eigene:7_Segment_SMD" (id 2) (at 208.28 71.12 0)
       (effects (font (size 1.27 1.27)) hide)
     )
@@
     (property "Reference" "AFF410" (id 0) (at 208.28 141.0802 0))
     (property "Value" "LTS-6980HR" (id 1) (at 208.28 143.6171 0))
-    (property "Footprint" "Display_7Segment:7SegmentLED_LTS6760_LTS6780" (id 2) (at 208.28 172.72 0)
+    (property "Footprint" "eigene:7_Segment_SMD" (id 2) (at 208.28 172.72 0)
       (effects (font (size 1.27 1.27)) hide)
     )
@@
     (property "Reference" "AFF413" (id 0) (at 340.36 19.1602 0))
     (property "Value" "LTS-6980HR" (id 1) (at 340.36 21.6971 0))
-    (property "Footprint" "Display_7Segment:7SegmentLED_LTS6760_LTS6780" (id 2) (at 340.36 50.8 0)
+    (property "Footprint" "eigene:7_Segment_SMD" (id 2) (at 340.36 50.8 0)
       (effects (font (size 1.27 1.27)) hide)
     )
@@
     (property "Reference" "AFF414" (id 0) (at 340.36 44.5602 0))
     (property "Value" "LTS-6980HR" (id 1) (at 340.36 47.0971 0))
-    (property "Footprint" "Display_7Segment:7SegmentLED_LTS6760_LTS6780" (id 2) (at 340.36 76.2 0)
+    (property "Footprint" "eigene:7_Segment_SMD" (id 2) (at 340.36 76.2 0)
       (effects (font (size 1.27 1.27)) hide)
     )
@@
     (property "Reference" "AFF419" (id 0) (at 340.36 171.5602 0))
     (property "Value" "LTS-6980HR" (id 1) (at 340.36 174.0971 0))
-    (property "Footprint" "Display_7Segment:7SegmentLED_LTS6760_LTS6780" (id 2) (at 340.36 203.2 0)
+    (property "Footprint" "eigene:7_Segment_SMD" (id 2) (at 340.36 203.2 0)
       (effects (font (size 1.27 1.27)) hide)
     )
@@
     (property "Reference" "AFF405" (id 0) (at 102.87 90.2802 0))
     (property "Value" "LTS-6980HR" (id 1) (at 102.87 92.8171 0))
-    (property "Footprint" "Display_7Segment:7SegmentLED_LTS6760_LTS6780" (id 2) (at 102.87 121.92 0)
+    (property "Footprint" "eigene:7_Segment_SMD" (id 2) (at 102.87 121.92 0)
       (effects (font (size 1.27 1.27)) hide)
     )
@@
     (property "Reference" "AFF417" (id 0) (at 340.36 120.7602 0))
     (property "Value" "LTS-6980HR" (id 1) (at 340.36 123.2971 0))
-    (property "Footprint" "Display_7Segment:7SegmentLED_LTS6760_LTS6780" (id 2) (at 340.36 152.4 0)
+    (property "Footprint" "eigene:7_Segment_SMD" (id 2) (at 340.36 152.4 0)
       (effects (font (size 1.27 1.27)) hide)
     )
@@
     (property "Reference" "AFF411" (id 0) (at 102.87 166.4802 0))
     (property "Value" "LTS-6980HR" (id 1) (at 102.87 169.0171 0))
-    (property "Footprint" "Display_7Segment:7SegmentLED_LTS6760_LTS6780" (id 2) (at 102.87 198.12 0)
+    (property "Footprint" "eigene:7_Segment_SMD" (id 2) (at 102.87 198.12 0)
       (effects (font (size 1.27 1.27)) hide)
     )
@@
     (property "Reference" "AFF406" (id 0) (at 208.28 90.2802 0))
     (property "Value" "LTS-6980HR" (id 1) (at 208.28 92.8171 0))
-    (property "Footprint" "Display_7Segment:7SegmentLED_LTS6760_LTS6780" (id 2) (at 208.28 121.92 0)
+    (property "Footprint" "eigene:7_Segment_SMD" (id 2) (at 208.28 121.92 0)
       (effects (font (size 1.27 1.27)) hide)
     )
@@
     (property "Reference" "AFF409" (id 0) (at 102.87 141.0802 0))
     (property "Value" "LTS-6980HR" (id 1) (at 102.87 143.6171 0))
-    (property "Footprint" "Display_7Segment:7SegmentLED_LTS6760_LTS6780" (id 2) (at 102.87 172.72 0)
+    (property "Footprint" "eigene:7_Segment_SMD" (id 2) (at 102.87 172.72 0)
       (effects (font (size 1.27 1.27)) hide)
     )
@@
     (property "Reference" "AFF416" (id 0) (at 340.36 95.3602 0))
     (property "Value" "LTS-6980HR" (id 1) (at 340.36 97.8971 0))
-    (property "Footprint" "Display_7Segment:7SegmentLED_LTS6760_LTS6780" (id 2) (at 340.36 127 0)
+    (property "Footprint" "eigene:7_Segment_SMD" (id 2) (at 340.36 127 0)
       (effects (font (size 1.27 1.27)) hide)
     )
@@
     (property "Reference" "AFF415" (id 0) (at 340.36 69.9602 0))
     (property "Value" "LTS-6980HR" (id 1) (at 340.36 72.4971 0))
-    (property "Footprint" "Display_7Segment:7SegmentLED_LTS6760_LTS6780" (id 2) (at 340.36 101.6 0)
+    (property "Footprint" "eigene:7_Segment_SMD" (id 2) (at 340.36 101.6 0)
       (effects (font (size 1.27 1.27)) hide)
     )
@@
     (property "Reference" "AFF408" (id 0) (at 208.28 115.6802 0))
     (property "Value" "LTS-6980HR" (id 1) (at 208.28 118.2171 0))
-    (property "Footprint" "Display_7Segment:7SegmentLED_LTS6760_LTS6780" (id 2) (at 208.28 147.32 0)
+    (property "Footprint" "eigene:7_Segment_SMD" (id 2) (at 208.28 147.32 0)
       (effects (font (size 1.27 1.27)) hide)
     )
@@
     (property "Reference" "AFF404" (id 0) (at 208.28 64.8802 0))
     (property "Value" "LTS-6980HR" (id 1) (at 208.28 67.4171 0))
-    (property "Footprint" "Display_7Segment:7SegmentLED_LTS6760_LTS6780" (id 2) (at 208.28 96.52 0)
+    (property "Footprint" "eigene:7_Segment_SMD" (id 2) (at 208.28 96.52 0)
       (effects (font (size 1.27 1.27)) hide)
     )
@@
     (property "Reference" "AFF401" (id 0) (at 102.87 39.4802 0))
     (property "Value" "LTS-6980HR" (id 1) (at 102.87 42.0171 0))
-    (property "Footprint" "Display_7Segment:7SegmentLED_LTS6760_LTS6780" (id 2) (at 102.87 71.12 0)
+    (property "Footprint" "eigene:7_Segment_SMD" (id 2) (at 102.87 71.12 0)
       (effects (font (size 1.27 1.27)) hide)
     )
@@
     (property "Reference" "AFF412" (id 0) (at 208.28 166.4802 0))
     (property "Value" "LTS-6980HR" (id 1) (at 208.28 169.0171 0))
-    (property "Footprint" "Display_7Segment:7SegmentLED_LTS6760_LTS6780" (id 2) (at 208.28 198.12 0)
+    (property "Footprint" "eigene:7_Segment_SMD" (id 2) (at 208.28 198.12 0)
       (effects (font (size 1.27 1.27)) hide)
     )
@@
     (property "Reference" "AFF418" (id 0) (at 340.36 146.1602 0))
     (property "Value" "LTS-6980HR" (id 1) (at 340.36 148.6971 0))
-    (property "Footprint" "Display_7Segment:7SegmentLED_LTS6760_LTS6780" (id 2) (at 340.36 177.8 0)
+    (property "Footprint" "eigene:7_Segment_SMD" (id 2) (at 340.36 177.8 0)
       (effects (font (size 1.27 1.27)) hide)
     )
@@
     (property "Reference" "AFF403" (id 0) (at 102.87 64.8802 0))
     (property "Value" "LTS-6980HR" (id 1) (at 102.87 67.4171 0))
-    (property "Footprint" "Display_7Segment:7SegmentLED_LTS6760_LTS6780" (id 2) (at 102.87 96.52 0)
+    (property "Footprint" "eigene:7_Segment_SMD" (id 2) (at 102.87 96.52 0)
       (effects (font (size 1.27 1.27)) hide)
     )
@@
     (property "Reference" "AFF420" (id 0) (at 340.36 196.9602 0))
     (property "Value" "LTS-6980HR" (id 1) (at 340.36 199.4971 0))
-    (property "Footprint" "Display_7Segment:7SegmentLED_LTS6760_LTS6780" (id 2) (at 340.36 228.6 0)
+    (property "Footprint" "eigene:7_Segment_SMD" (id 2) (at 340.36 228.6 0)
       (effects (font (size 1.27 1.27)) hide)
     )
@@
     (property "Reference" "AFF407" (id 0) (at 102.87 115.6802 0))
     (property "Value" "LTS-6980HR" (id 1) (at 102.87 118.2171 0))
-    (property "Footprint" "Display_7Segment:7SegmentLED_LTS6760_LTS6780" (id 2) (at 102.87 147.32 0)
-      (effects (font (size 1.27 1.27)) hide)
-    )
+    (property "Footprint" "eigene:7_Segment_SMD" (id 2) (at 102.87 147.32 0)
+      (effects (font (size 1.27 1.27)) hide)
+    )

Commit message: update
Other:
- note added: "157112S12700"
Changed lines of the file:
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@@
     (stroke (width 0) (type default) (color 0 0 0 0))
+  )
+  (text "157112S12700 " (at 95.25 30.48 0)
+    (effects (font (size 1.27 1.27)) (justify left bottom))
   )
   (hierarchical_label "CLK" (shape input) (at 27.94 210.82 180)

Commit message: finalize initial routing
Connections:
- net at AFF413.1 (e): now also AFF414.1 (e), AFF415.1 (e), AFF416.1 (e), AFF417.1 (e), AFF418.1 (e), AFF419.1 (e), AFF420.1 (e), U405.21 (SEG_E)
- net at AFF413.10 (g): now also AFF414.10 (g), AFF415.10 (g), AFF416.10 (g), AFF417.10 (g), AFF418.10 (g), AFF419.10 (g), AFF420.10 (g), U405.17 (SEG_G)
- net at AFF413.2 (d): now also AFF414.2 (d), AFF415.2 (d), AFF416.2 (d), AFF417.2 (d), AFF418.2 (d), AFF419.2 (d), AFF420.2 (d), U405.23 (SEG_D)
- net at AFF413.4 (c): now also AFF414.4 (c), AFF415.4 (c), AFF416.4 (c), AFF417.4 (c), AFF418.4 (c), AFF419.4 (c), AFF420.4 (c), U405.20 (SEG_C)
- net at AFF413.5 (DP), AFF414.5 (DP), AFF415.5 (DP)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: now also AFF416.5 (DP), AFF417.5 (DP), AFF418.5 (DP), AFF419.5 (DP), AFF420.5 (DP)
- net at AFF413.6 (b): now also AFF414.6 (b), AFF415.6 (b), AFF416.6 (b), AFF417.6 (b), AFF418.6 (b), AFF419.6 (b), AFF420.6 (b), U405.16 (SEG_B)
- net at AFF413.7 (a): now also AFF414.7 (a), AFF415.7 (a), AFF416.7 (a), AFF417.7 (a), AFF418.7 (a), AFF419.7 (a), AFF420.7 (a), U405.14 (SEG_A)
- net at AFF413.9 (f): now also AFF414.9 (f), AFF415.9 (f), AFF416.9 (f), AFF417.9 (f), AFF418.9 (f), AFF419.9 (f), AFF420.9 (f), U405.15 (SEG_F)
