File: hardware/cpu.kicad_sch (KiCad schematic)
At the start: 84 parts, among them J1 Jack-DC, J2 DCF77 Antenna, J3 SWD, J4 USB_B, Q14 BSS138, Q15 BSS138, Q16 BSS138, U7 AZ1117-3.3, U8 L7805, U9 STM32F103C8Tx, Y1 32.768kHz, Y2 8MHz

Commit message: start layout, finalize schematic
Parts:
- added Q508: BC856, Package_TO_SOT_SMD:SOT-23, symbol Transistor_BJT:BC856
- added Q511: BSS138, Package_TO_SOT_SMD:SOT-23, symbol Transistor_FET:BSS138
- added R525, R527, R537: 100k, Resistor_SMD:R_0805_2012Metric, symbol Device:R
- added R535, R536: 10k, Resistor_SMD:R_0805_2012Metric, symbol Device:R
- C501: renamed from C28; footprint (none) -> Capacitor_SMD:CP_Elec_10x10.5
- C502: renamed from C26; footprint (none) -> Capacitor_SMD:C_0805_2012Metric
- C503: renamed from C9; footprint (none) -> Capacitor_SMD:C_0805_2012Metric
- C504: renamed from C13; footprint (none) -> Capacitor_SMD:C_0805_2012Metric
- C505: renamed from C15; footprint (none) -> Capacitor_SMD:C_0805_2012Metric
- C506: renamed from C19; footprint (none) -> Capacitor_SMD:C_0805_2012Metric
- C507: renamed from C20; footprint (none) -> Capacitor_SMD:C_0805_2012Metric
- C508: renamed from C25; footprint (none) -> Capacitor_SMD:C_0805_2012Metric
- C509: renamed from C23; footprint (none) -> Capacitor_SMD:C_0805_2012Metric
- C510: renamed from C24; footprint (none) -> Capacitor_SMD:C_0805_2012Metric
- C511: renamed from C21; footprint (none) -> Capacitor_SMD:C_0805_2012Metric
- C512: renamed from C22; footprint (none) -> Capacitor_SMD:C_0805_2012Metric
- C513: renamed from C8; footprint (none) -> Capacitor_SMD:C_0805_2012Metric
- C514: renamed from C11; footprint (none) -> Capacitor_SMD:C_0805_2012Metric
- C515: renamed from C16; footprint (none) -> Capacitor_SMD:C_0805_2012Metric
- C516: renamed from C18; footprint (none) -> Capacitor_SMD:C_0805_2012Metric
- C517: renamed from C29; footprint (none) -> Capacitor_SMD:C_0805_2012Metric
- C518: renamed from C27; footprint (none) -> Capacitor_SMD:C_0805_2012Metric
- C519, C520, C526: renamed from C?; footprint (none) -> Capacitor_SMD:C_0805_2012Metric
- C521: renamed from C7; footprint (none) -> Capacitor_SMD:C_0805_2012Metric
- C522: renamed from C10; footprint (none) -> Capacitor_SMD:C_0805_2012Metric
- C523: renamed from C12; footprint (none) -> Capacitor_SMD:C_0805_2012Metric
- C524: renamed from C14; footprint (none) -> Capacitor_SMD:C_0805_2012Metric
- C525: renamed from C17; footprint (none) -> Capacitor_SMD:C_0805_2012Metric
- D501: renamed from D133; footprint (none) -> Diode_SMD:D_MiniMELF
- D503: renamed from D134; footprint (none) -> LED_SMD:LED_0603_1608Metric
- D504: renamed from D132; footprint (none) -> LED_SMD:LED_0603_1608Metric
- FB501: renamed from FB1; footprint (none) -> Resistor_SMD:R_4020_10251Metric
- FB502: renamed from FB2; footprint (none) -> Resistor_SMD:R_4020_10251Metric
- J501: renamed from J1; footprint (none) -> Connector_BarrelJack:BarrelJack_Horizontal
- J502: renamed from J2; footprint (none) -> Connector_PinHeader_2.54mm:PinHeader_1x04_P2.54mm_Vertical
- J503: renamed from J3; footprint (none) -> Connector_PinHeader_2.54mm:PinHeader_1x04_P2.54mm_Horizontal
- J504: renamed from J4; footprint (none) -> Connector_USB:USB_B_OST_USB-B1HSxx_Horizontal
- R501, R502, R504, R506, R508, R509, R511, R512, R513, R514, R515, R518, R519, R520, R521, R522, R530, R531, R534: renamed from R?; footprint (none) -> Resistor_SMD:R_0805_2012Metric
- R503: renamed from R49; footprint (none) -> Resistor_SMD:R_0805_2012Metric
- R505: renamed from R53; footprint (none) -> Resistor_SMD:R_0805_2012Metric
- R507: renamed from R51; footprint (none) -> Resistor_SMD:R_0805_2012Metric
- R510: renamed from R52; footprint (none) -> Resistor_SMD:R_0805_2012Metric
- R516: renamed from R44; footprint (none) -> Resistor_SMD:R_0805_2012Metric
- R517: renamed from R45; footprint (none) -> Resistor_SMD:R_0805_2012Metric
- R523: renamed from R46; footprint (none) -> Resistor_SMD:R_0805_2012Metric
- R524: renamed from R56; footprint (none) -> Resistor_SMD:R_0805_2012Metric
- R526: renamed from R50; footprint (none) -> Resistor_SMD:R_0805_2012Metric
- R528: renamed from R47; footprint (none) -> Resistor_SMD:R_0805_2012Metric
- R529: renamed from R54; footprint (none) -> Resistor_SMD:R_0805_2012Metric
- R532: renamed from R55; footprint (none) -> Resistor_SMD:R_0805_2012Metric
- R533: renamed from R48; footprint (none) -> Resistor_SMD:R_0805_2012Metric
- U501: renamed from U8; footprint (none) -> Package_TO_SOT_SMD:TO-252-2
- U502: renamed from U7; footprint (none) -> Package_TO_SOT_SMD:SOT-223-3_TabPin2
- Y501: renamed from Y2; footprint (none) -> Crystal:Crystal_SMD_HC49-SD
- Y502: renamed from Y1; footprint (none) -> Crystal:Crystal_SMD_SeikoEpson_MC306-4Pin_8.0x3.2mm
- gave numbers to parts that had none: 9
- renumbered Q14 to Q505, Q16 to Q509, Q15 to Q510, U9 to U503
Connections:
- net +3V3: now also Q508.2 (E), R525.2; no longer R530.2
- net +5V: now also R535.2
- net GND: now also Q511.2 (S), R537.2
- net at U503.14 (PA4): now also R536.1
- net /Disconnect: now reaches U503.45 (PB8)
- net /Disconnect: now also R527.1
- new net: Q508.1 (B), R525.1, R527.2
- new net: Q508.3 (C), R530.2
- new net: Q511.1 (G), R536.2, R537.1
- new net: Q511.3 (D), R535.1
- no-connect marks 17 -> 15
Other:
- moved on the sheet: J502, Q505, R516, R517

Commit message: update Layout
Other:
- moved on the sheet: C513, C514, C515, C516, U502

Commit message: update Schematic
Parts:
- Y502: symbol Device:Crystal -> Device:Crystal_GND23
Connections:
- net at C511.1, U503.3 (PC14): now also Y502.4; no longer Y502.2
Changed lines of the file:
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@@
     (pin "2")
   )
-  (symbol (lib_id "Device:Crystal") (at 148.59 82.55 90) (unit 1)
-    (in_bom yes) (on_board yes) (fields_autoplaced)
-    (property "Reference" "Y502" (id 0) (at 151.9174 81.7153 90)
+  (symbol (lib_id "Device:Crystal_GND23") (at 148.59 82.55 90) (unit 1)
+    (in_bom yes) (on_board yes)
+    (property "Reference" "Y502" (id 0) (at 153.67 80.01 90)
       (effects (font (size 1.27 1.27)) (justify right))
     )
-    (property "Value" "32.768kHz" (id 1) (at 151.9174 84.2522 90)
+    (property "Value" "32.768kHz" (id 1) (at 152.4 85.09 90)
       (effects (font (size 1.27 1.27)) (justify right))
     )
@@
     (pin "1")
     (pin "2")
+    (pin "3")
+    (pin "4")
   )
   (symbol (lib_id "Device:C_Polarized") (at 220.98 34.29 0) (unit 1)

Commit message: update
Parts:
- C503, C517: footprint Capacitor_SMD:C_0805_2012Metric -> Capacitor_SMD:CP_Elec_5x5.8
- C518: value C -> 100n
- FB501, FB502: footprint Resistor_SMD:R_4020_10251Metric -> eigene:SMB-001
Connections:
- net +3.3V is gone; now on net +3V3: C518.1, D501.2 (A), J502.4 (Pin_4), J503.1 (Pin_1), Q504.1 (G), Q506.1 (G), R503.2, R513.2, R519.2, R523.1, U503.24 (VDD), U503.36 (VDD), U503.48 (VDD), U503.9 (VDDA)
- net at C511.1, U503.3 (PC14): now also Y502.1; no longer Y502.4
- net at C512.1, U503.4 (PC15): now also Y502.4; no longer Y502.1
Other:
- note added: "EEE-FT1C101AR"
- moved on the sheet: Y502

Commit message: update
Connections:
- net +3V3: no longer C521.1
- net +5V: now also C521.1, D504.2 (A); no longer R526.2
- net at R526.1: now also Q510.3 (D); no longer D504.2 (A)
- net at D504.1 (K): now also R526.2; no longer Q510.3 (D)
Other:
- moved on the sheet: D504, R526

Commit message: finalize initial routing
Connections:
- net /CS_Date: now also Q503.3 (D), R511.1
- net /CS_Inner: now also Q502.3 (D), R506.1
- net /CS_Outer: now also Q501.3 (D), R501.1
- net /CS_Time: now also Q507.3 (D), R518.1
- net /CS_pulse: now also Q511.3 (D), R535.1
Changed lines of the file:
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@@
   (junction (at 193.04 45.72) (diameter 0) (color 0 0 0 0)
   )
+  (junction (at 266.7 25.4) (diameter 0) (color 0 0 0 0)
+  )
   (junction (at 137.16 99.06) (diameter 0) (color 0 0 0 0)
   )
@@
   (junction (at 195.58 45.72) (diameter 0) (color 0 0 0 0)
   )
+  (junction (at 266.7 113.03) (diameter 0) (color 0 0 0 0)
+  )
   (junction (at 241.3 114.3) (diameter 0) (color 0 0 0 0)
   )
@@
   (junction (at 266.7 35.56) (diameter 0) (color 0 0 0 0)
   )
+  (junction (at 266.7 54.61) (diameter 0) (color 0 0 0 0)
+  )
   (junction (at 50.8 35.56) (diameter 0) (color 0 0 0 0)
   )
@@
   (junction (at 209.55 29.21) (diameter 0) (color 0 0 0 0)
   )
+  (junction (at 266.7 144.78) (diameter 0) (color 0 0 0 0)
+  )
   (junction (at 16.51 190.5) (diameter 0) (color 0 0 0 0)
   )
@@
   )
   (junction (at 50.8 177.8) (diameter 0) (color 0 0 0 0)
+  )
+  (junction (at 266.7 83.82) (diameter 0) (color 0 0 0 0)
   )
   (junction (at 259.08 118.11) (diameter 0) (color 0 0 0 0)
@@
     (stroke (width 0) (type default) (color 0 0 0 0))
   )
-  (wire (pts (xy 266.7 85.09) (xy 270.51 85.09))
+  (wire (pts (xy 266.7 83.82) (xy 270.51 83.82))
     (stroke (width 0) (type default) (color 0 0 0 0))
   )
@@
     (stroke (width 0) (type default) (color 0 0 0 0))
   )
+  (wire (pts (xy 266.7 144.78) (xy 270.51 144.78))
+    (stroke (width 0) (type default) (color 0 0 0 0))
+  )
   (wire (pts (xy 187.96 49.53) (xy 187.96 29.21))
     (stroke (width 0) (type default) (color 0 0 0 0))
@@
     (stroke (width 0) (type default) (color 0 0 0 0))
   )
-  (wire (pts (xy 266.7 26.67) (xy 270.51 26.67))
+  (wire (pts (xy 266.7 25.4) (xy 270.51 25.4))
     (stroke (width 0) (type default) (color 0 0 0 0))
   )
@@
     (stroke (width 0) (type default) (color 0 0 0 0))
   )
-  (wire (pts (xy 266.7 114.3) (xy 270.51 114.3))
+  (wire (pts (xy 266.7 113.03) (xy 270.51 113.03))
     (stroke (width 0) (type default) (color 0 0 0 0))
   )
@@
     (stroke (width 0) (type default) (color 0 0 0 0))
   )
-  (wire (pts (xy 266.7 55.88) (xy 270.51 55.88))
+  (wire (pts (xy 266.7 54.61) (xy 270.51 54.61))
     (stroke (width 0) (type default) (color 0 0 0 0))
   )
@@
   )
   (wire (pts (xy 208.28 107.95) (xy 213.36 107.95))
-    (stroke (width 0) (type default) (color 0 0 0 0))
-  )
-  (wire (pts (xy 266.7 146.05) (xy 270.51 146.05))
     (stroke (width 0) (type default) (color 0 0 0 0))
   )
@@
     (effects (font (size 1.27 1.27)) (justify left))
   )
-  (hierarchical_label "{slash}CS_pulse" (shape output) (at 270.51 146.05 0)
+  (hierarchical_label "{slash}CS_pulse" (shape output) (at 270.51 144.78 0)
     (effects (font (size 1.27 1.27)) (justify left))
   )
@@
     (effects (font (size 1.27 1.27)) (justify left))
   )
-  (hierarchical_label "{slash}CS_Date" (shape output) (at 270.51 85.09 0)
-    (effects (font (size 1.27 1.27)) (justify left))
-  )
-  (hierarchical_label "{slash}CS_Time" (shape output) (at 270.51 114.3 0)
-    (effects (font (size 1.27 1.27)) (justify left))
-  )
-  (hierarchical_label "{slash}CS_Inner" (shape output) (at 270.51 55.88 0)
-    (effects (font (size 1.27 1.27)) (justify left))
-  )
-  (hierarchical_label "{slash}CS_Outer" (shape output) (at 270.51 26.67 0)
+  (hierarchical_label "{slash}CS_Date" (shape output) (at 270.51 83.82 0)
+    (effects (font (size 1.27 1.27)) (justify left))
+  )
+  (hierarchical_label "{slash}CS_Time" (shape output) (at 270.51 113.03 0)
+    (effects (font (size 1.27 1.27)) (justify left))
+  )
+  (hierarchical_label "{slash}CS_Inner" (shape output) (at 270.51 54.61 0)
+    (effects (font (size 1.27 1.27)) (justify left))
+  )
+  (hierarchical_label "{slash}CS_Outer" (shape output) (at 270.51 25.4 0)
     (effects (font (size 1.27 1.27)) (justify left))
   )
@@
   (symbol (lib_id "power:+5V") (at 16.51 176.53 0) (unit 1)
     (in_bom yes) (on_board yes) (fields_autoplaced)
-    (property "Reference" "#PWR?" (id 0) (at 16.51 180.34 0)
+    (property "Reference" "#PWR0109" (id 0) (at 16.51 180.34 0)
       (effects (font (size 1.27 1.27)) hide)
     )
