File: hardware/dcf77.kicad_sch (KiCad schematic)
At the start: 0 parts

Commit message: start layout, finalize schematic
Other:
- sheet CPU ports: added /CS_pulse; removed none
- sheet Status_LEDs ports: added /CS_pulse; removed none
