File: hardware/review/Status.kicad_sch (KiCad schematic)
At the start: 97 parts, among them Q401 BSS138, Q402 BSS138, Q403 BSS138, Q404 BSS138, Q405 BSS138, Q406 BSS138, Q407 BSS138, Q408 BSS138, Q409 BSS138, Q410 BSS138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

Commit message: update resistor values in Schematic and BOM Bugfix in Code added test stand
Parts:
- R401, R402, R403, R404, R405, R406, R407, R408, R409, R410, R411, R412, R413: value R -> 2k2
- R427, R428, R442: value 20k -> 10k
Changed lines of the file:
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@@
       (effects (font (size 1.27 1.27)) (justify left))
     )
-    (property "Value" "R" (id 1) (at 133.858 320.4722 0)
+    (property "Value" "2k2" (id 1) (at 133.858 320.4722 0)
       (effects (font (size 1.27 1.27)) (justify left))
     )
@@
       (effects (font (size 1.27 1.27)) (justify left))
     )
-    (property "Value" "R" (id 1) (at 80.518 320.4722 0)
+    (property "Value" "2k2" (id 1) (at 80.518 320.4722 0)
       (effects (font (size 1.27 1.27)) (justify left))
     )
@@
       (effects (font (size 1.27 1.27)) (justify left))
     )
-    (property "Value" "R" (id 1) (at 89.408 320.4722 0)
+    (property "Value" "2k2" (id 1) (at 89.408 320.4722 0)
       (effects (font (size 1.27 1.27)) (justify left))
     )
@@
       (effects (font (size 1.27 1.27)) (justify left))
     )
-    (property "Value" "R" (id 1) (at 44.958 320.4722 0)
+    (property "Value" "2k2" (id 1) (at 44.958 320.4722 0)
       (effects (font (size 1.27 1.27)) (justify left))
     )
@@
       (effects (font (size 1.27 1.27)) (justify left))
     )
-    (property "Value" "R" (id 1) (at 116.078 320.4722 0)
+    (property "Value" "2k2" (id 1) (at 116.078 320.4722 0)
       (effects (font (size 1.27 1.27)) (justify left))
     )
@@
       (effects (font (size 1.27 1.27)) (justify left))
     )
-    (property "Value" "R" (id 1) (at 142.748 320.4722 0)
+    (property "Value" "2k2" (id 1) (at 142.748 320.4722 0)
       (effects (font (size 1.27 1.27)) (justify left))
     )
@@
       (effects (font (size 1.27 1.27)) (justify left))
     )
-    (property "Value" "R" (id 1) (at 53.848 320.4722 0)
+    (property "Value" "2k2" (id 1) (at 53.848 320.4722 0)
       (effects (font (size 1.27 1.27)) (justify left))
     )
@@
       (effects (font (size 1.27 1.27)) (justify left))
     )
-    (property "Value" "R" (id 1) (at 124.968 320.4722 0)
+    (property "Value" "2k2" (id 1) (at 124.968 320.4722 0)
       (effects (font (size 1.27 1.27)) (justify left))
     )
@@
       (effects (font (size 1.27 1.27)) (justify left))
     )
-    (property "Value" "20k" (id 1) (at 146.558 168.0722 0)
+    (property "Value" "10k" (id 1) (at 146.558 168.0722 0)
       (effects (font (size 1.27 1.27)) (justify left))
     )
@@
       (effects (font (size 1.27 1.27)) (justify left))
     )
-    (property "Value" "R" (id 1) (at 71.628 320.4722 0)
+    (property "Value" "2k2" (id 1) (at 71.628 320.4722 0)
       (effects (font (size 1.27 1.27)) (justify left))
     )
@@
       (effects (font (size 1.27 1.27)) (justify left))
     )
-    (property "Value" "20k" (id 1) (at 278.638 198.5522 0)
+    (property "Value" "10k" (id 1) (at 278.638 198.5522 0)
       (effects (font (size 1.27 1.27)) (justify left))
     )
@@
       (effects (font (size 1.27 1.27)) (justify left))
     )
-    (property "Value" "R" (id 1) (at 98.298 320.4722 0)
+    (property "Value" "2k2" (id 1) (at 98.298 320.4722 0)
       (effects (font (size 1.27 1.27)) (justify left))
     )
@@
       (effects (font (size 1.27 1.27)) (justify left))
     )
-    (property "Value" "R" (id 1) (at 107.188 320.4722 0)
+    (property "Value" "2k2" (id 1) (at 107.188 320.4722 0)
       (effects (font (size 1.27 1.27)) (justify left))
     )
@@
       (effects (font (size 1.27 1.27)) (justify left))
     )
-    (property "Value" "R" (id 1) (at 151.638 320.4722 0)
+    (property "Value" "2k2" (id 1) (at 151.638 320.4722 0)
       (effects (font (size 1.27 1.27)) (justify left))
     )
@@
       (effects (font (size 1.27 1.27)) (justify left))
     )
-    (property "Value" "20k" (id 1) (at 41.148 168.0722 0)
+    (property "Value" "10k" (id 1) (at 41.148 168.0722 0)
       (effects (font (size 1.27 1.27)) (justify left))
     )
@@
       (effects (font (size 1.27 1.27)) (justify left))
     )
-    (property "Value" "R" (id 1) (at 62.738 320.4722 0)
-      (effects (font (size 1.27 1.27)) (justify left))
-    )
+    (property "Value" "2k2" (id 1) (at 62.738 320.4722 0)
+      (effects (font (size 1.27 1.27)) (justify left))
+    )
