File: hardware/review/cpu.kicad_sch (KiCad schematic)
At the start: 92 parts, among them J501 Jack-DC, J502 DCF77 Antenna, J503 SWD, J504 USB_B, Q501 BSS138, Q502 BSS138, Q503 BSS138, Q504 BSS138, Q505 BSS138, Q506 BSS138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

Commit message: update resistor values in Schematic and BOM Bugfix in Code added test stand
Parts:
- C511, C512: value 20p -> 10p
- R524: value 1k -> 2k2
- U501: footprint Package_TO_SOT_SMD:TO-252-2 -> Package_TO_SOT_SMD:TO-263-2
Changed lines of the file:
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@@
     (property "Reference" "U501" (id 0) (at 92.71 29.9552 0))
     (property "Value" "L7805" (id 1) (at 92.71 32.4921 0))
-    (property "Footprint" "Package_TO_SOT_SMD:TO-252-2" (id 2) (at 93.345 39.37 0)
+    (property "Footprint" "Package_TO_SOT_SMD:TO-263-2" (id 2) (at 93.345 39.37 0)
       (effects (font (size 1.27 1.27) italic) (justify left) hide)
     )
@@
     (in_bom yes) (on_board yes)
     (property "Reference" "C512" (id 0) (at 133.35 85.09 90))
-    (property "Value" "20p" (id 1) (at 140.97 85.09 90))
+    (property "Value" "10p" (id 1) (at 140.97 85.09 90))
     (property "Footprint" "Capacitor_SMD:C_0805_2012Metric" (id 2) (at 133.35 87.3252 0)
       (effects (font (size 1.27 1.27)) hide)
@@
     (in_bom yes) (on_board yes)
     (property "Reference" "C511" (id 0) (at 133.35 77.47 90))
-    (property "Value" "20p" (id 1) (at 140.97 77.47 90))
+    (property "Value" "10p" (id 1) (at 140.97 77.47 90))
     (property "Footprint" "Capacitor_SMD:C_0805_2012Metric" (id 2) (at 133.35 79.7052 0)
       (effects (font (size 1.27 1.27)) hide)
@@
       (effects (font (size 1.27 1.27)) (justify right))
     )
-    (property "Value" "1k" (id 1) (at 239.268 132.5122 0)
-      (effects (font (size 1.27 1.27)) (justify right))
-    )
+    (property "Value" "2k2" (id 1) (at 239.268 132.5122 0)
+      (effects (font (size 1.27 1.27)) (justify right))
+    )
